File: PCB/ESP32_Atmega328/ESP32_Atmega328.kicad_sch (KiCad schematic)
At the start: 25 parts

Commit message: Added parts, rerouted some, added component zips
Parts:
- removed SW1: (no value), symbol Switch:SW_SPDT
- added C7, C8: 100n, Capacitor_SMD:C_0603_1608Metric, symbol Device:C_Small
- added J4: (no value), symbol U.FL-R-SMT_01_:U.FL-R-SMT(01)
- added J5: (no value), symbol Connector_Generic:Conn_01x02
- added J6: (no value), symbol Connector_Generic:Conn_01x05
- added J7: (no value), Connector_PinHeader_2.54mm:PinHeader_1x02_P2.54mm_Vertical, symbol Connector_Generic:Conn_01x02
- added JP1: (no value), symbol Jumper:Jumper_2_Open
- ATM328P1: footprint (none) -> Package_QFP:TQFP-32_7x7mm_P0.8mm
- BT1: value (none) -> S8421-45R; footprint (none) -> footprints:BAT_S8421-45R
- C3, C6: value (none) -> 1u
- C5: value (none) -> 100n
- D1: value (none) -> 1N4148; footprint Diode_THT:D_DO-35_SOD27_P7.62mm_Horizontal -> (none)
- D2: value (none) -> BLUE; footprint (none) -> LED_SMD:LED_0603_1608Metric
- J1: value (none) -> ESP_CONN; footprint Connector_JST:JST_EH_B4B-EH-A_1x04_P2.50mm_Vertical -> (none)
- PWR1: value (none) -> MCP1700-3002E_SOT23
- R3: value (none) -> 10k; footprint (none) -> Resistor_SMD:R_0603_1608Metric
- R4: value (none) -> 1k5; footprint (none) -> Resistor_SMD:R_0603_1608Metric
- RFM95W1: footprint (none) -> footprints:XCVR_RFM95W-915S2
Connections:
- net +3V3: now also ATM328P1.18 (AVCC), C7.1, J7.1 (Pin_1), JP1.1 (A); no longer D2.2 (A)
- net +6V: now also C3.1, PWR1.3 (VI)
- net GND: now also C7.2, C8.2, J4.1 (GND), J4.2 (GND), J7.2 (Pin_2)
- net RFM_ANT: now reaches RFM95W1.9 (ANT)
- net RFM_ANT: now also J4.3 (SIG)
- net PD7: now reaches ATM328P1.11 (PD7)
- net PD7: now also J6.1 (Pin_1)
- net PB0: now reaches ATM328P1.12 (PB0)
- net PB0: now also J6.5 (Pin_5)
- net at ATM328P1.20 (AREF): now also C8.1
- net PC0: now reaches ATM328P1.23 (PC0)
- net PC0: now also J6.4 (Pin_4)
- net PC1: now reaches ATM328P1.24 (PC1)
- net PC1: now also J6.3 (Pin_3)
- net PC2: now reaches ATM328P1.25 (PC2)
- net PC2: now also J6.2 (Pin_2)
- net CLOCK_SCL renamed I2C_SCL
- net I2C_SCL: now also J5.1 (Pin_1)
- net CLOCK_SDA renamed I2C_SDA
- net I2C_SDA: now also J5.2 (Pin_2)
- new net: D2.2 (A), JP1.2 (B)
- no-connect marks 18 -> 10
Other:
- moved on the sheet: ATM328P1, C1, C2, C3, D2, DS3231M1, J3, R1, R2, R4, RFM95W1

Commit message: Antenna impedance matching to 50ohms, and added more ground vias around the antenna connector
Parts:
- D1: footprint (none) -> Diode_SMD:D_SOD-323
- H1, H2, H3, H4: footprint MountingHole:MountingHole_4.3mm_M4_Pad_Via -> (none)
- J2: value (none) -> PWR_IN_CONN
- J3: value (none) -> PROG_CONN; footprint (none) -> Connector_JST:JST_XH_B5B-XH-A_1x05_P2.50mm_Vertical
- J4: value (none) -> U.FL-R-SMT(01); footprint (none) -> footprints:HRS_U.FL-R-SMT(01)
- J5: value (none) -> I2C_CONN; footprint (none) -> Connector_PinHeader_2.54mm:PinHeader_1x02_P2.54mm_Vertical
- J6: value (none) -> BREAKOUT_CONN; footprint (none) -> Connector_PinHeader_2.54mm:PinHeader_1x05_P2.54mm_Vertical
- J7: value (none) -> PWR_OUT_CONN
- JP1: value (none) -> Jumper_2_Open; footprint (none) -> Connector_PinHeader_2.54mm:PinHeader_1x02_P2.54mm_Vertical
Changed lines of the file:
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@@
       (effects (font (size 1.27 1.27)) (justify left))
     )
-    (property "Value" "" (id 1) (at 267.97 53.3399 0)
+    (property "Value" "PWR_OUT_CONN" (id 1) (at 267.97 53.3399 0)
       (effects (font (size 1.27 1.27)) (justify left))
     )
@@
       (effects (font (size 1.27 1.27)) (justify left))
     )
-    (property "Value" "" (id 1) (at 267.97 93.9799 0)
-      (effects (font (size 1.27 1.27)) (justify left))
-    )
-    (property "Footprint" "" (id 2) (at 265.43 92.71 0)
+    (property "Value" "BREAKOUT_CONN" (id 1) (at 267.97 93.9799 0)
+      (effects (font (size 1.27 1.27)) (justify left))
+    )
+    (property "Footprint" "Connector_PinHeader_2.54mm:PinHeader_1x05_P2.54mm_Vertical" (id 2) (at 265.43 92.71 0)
       (effects (font (size 1.27 1.27)) hide)
     )
@@
       (effects (font (size 1.27 1.27)) (justify left))
     )
-    (property "Value" "" (id 1) (at 267.97 78.7399 0)
-      (effects (font (size 1.27 1.27)) (justify left))
-    )
-    (property "Footprint" "" (id 2) (at 265.43 76.2 0)
+    (property "Value" "I2C_CONN" (id 1) (at 267.97 78.7399 0)
+      (effects (font (size 1.27 1.27)) (justify left))
+    )
+    (property "Footprint" "Connector_PinHeader_2.54mm:PinHeader_1x02_P2.54mm_Vertical" (id 2) (at 265.43 76.2 0)
       (effects (font (size 1.27 1.27)) hide)
     )
@@
       (effects (font (size 1.27 1.27)) (justify left))
     )
-    (property "Footprint" "MountingHole:MountingHole_4.3mm_M4_Pad_Via" (id 2) (at 259.08 34.29 0)
+    (property "Footprint" "" (id 2) (at 259.08 34.29 0)
       (effects (font (size 1.27 1.27)) hide)
     )
@@
       (effects (font (size 1.27 1.27)) (justify left))
     )
-    (property "Footprint" "MountingHole:MountingHole_4.3mm_M4_Pad_Via" (id 2) (at 259.08 27.94 0)
+    (property "Footprint" "" (id 2) (at 259.08 27.94 0)
       (effects (font (size 1.27 1.27)) hide)
     )
@@
     (in_bom yes) (on_board yes) (fields_autoplaced)
     (property "Reference" "JP1" (id 0) (at 114.3 170.18 0))
-    (property "Value" "" (id 1) (at 114.3 172.72 0))
-    (property "Footprint" "" (id 2) (at 114.3 176.53 0)
+    (property "Value" "Jumper_2_Open" (id 1) (at 114.3 172.72 0))
+    (property "Footprint" "Connector_PinHeader_2.54mm:PinHeader_1x02_P2.54mm_Vertical" (id 2) (at 114.3 176.53 0)
       (effects (font (size 1.27 1.27)) hide)
     )
@@
     (in_bom yes) (on_board yes) (fields_autoplaced)
     (property "Reference" "J4" (id 0) (at 165.4429 128.27 0))
-    (property "Value" "" (id 1) (at 165.4429 130.81 0))
-    (property "Footprint" "" (id 2) (at 163.83 137.16 0)
+    (property "Value" "U.FL-R-SMT(01)" (id 1) (at 165.4429 130.81 0))
+    (property "Footprint" "footprints:HRS_U.FL-R-SMT(01)" (id 2) (at 163.83 137.16 0)
       (effects (font (size 1.27 1.27)) (justify left bottom) hide)
     )
@@
       (effects (font (size 1.27 1.27)) (justify left))
     )
-    (property "Footprint" "" (id 2) (at 198.755 36.83 0)
+    (property "Footprint" "Diode_SMD:D_SOD-323" (id 2) (at 198.755 36.83 0)
       (effects (font (size 1.27 1.27)) hide)
     )
@@
       (effects (font (size 1.27 1.27)) (justify left))
     )
-    (property "Footprint" "MountingHole:MountingHole_4.3mm_M4_Pad_Via" (id 2) (at 259.08 40.64 0)
+    (property "Footprint" "" (id 2) (at 259.08 40.64 0)
       (effects (font (size 1.27 1.27)) hide)
     )
@@
       (effects (font (size 1.27 1.27)) (justify left))
     )
-    (property "Footprint" "MountingHole:MountingHole_4.3mm_M4_Pad_Via" (id 2) (at 259.08 21.59 0)
+    (property "Footprint" "" (id 2) (at 259.08 21.59 0)
       (effects (font (size 1.27 1.27)) hide)
     )
@@
       (effects (font (size 1.27 1.27)) (justify left))
     )
-    (property "Value" "" (id 1) (at 267.97 111.7599 0)
-      (effects (font (size 1.27 1.27)) (justify left))
-    )
-    (property "Footprint" "" (id 2) (at 265.43 110.49 0)
+    (property "Value" "PROG_CONN" (id 1) (at 267.97 111.7599 0)
+      (effects (font (size 1.27 1.27)) (justify left))
+    )
+    (property "Footprint" "Connector_JST:JST_XH_B5B-XH-A_1x05_P2.50mm_Vertical" (id 2) (at 265.43 110.49 0)
       (effects (font (size 1.27 1.27)) hide)
     )
@@
       (effects (font (size 1.27 1.27)) (justify left))
     )
-    (property "Value" "" (id 1) (at 31.75 156.2099 0)
+    (property "Value" "PWR_IN_CONN" (id 1) (at 31.75 156.2099 0)
       (effects (font (size 1.27 1.27)) (justify left))
     )
@@
     )
     (path "/e1315cf7-41f2-4028-9878-1b661c433c27"
-      (reference "H1") (unit 1) (value "MountingHole_Pad") (footprint "MountingHole:MountingHole_4.3mm_M4_Pad_Via")
+      (reference "H1") (unit 1) (value "MountingHole_Pad") (footprint "MountingHole:MountingHole_3.2mm_M3_Pad_Via")
     )
     (path "/94644b12-8e8f-4fb1-ba7e-f33b4b619430"
-      (reference "H2") (unit 1) (value "MountingHole_Pad") (footprint "MountingHole:MountingHole_4.3mm_M4_Pad_Via")
+      (reference "H2") (unit 1) (value "MountingHole_Pad") (footprint "MountingHole:MountingHole_3.2mm_M3_Pad_Via")
     )
     (path "/9291c528-baa9-455a-b63d-b146522fcd3e"
-      (reference "H3") (unit 1) (value "MountingHole_Pad") (footprint "MountingHole:MountingHole_4.3mm_M4_Pad_Via")
+      (reference "H3") (unit 1) (value "MountingHole_Pad") (footprint "MountingHole:MountingHole_3.2mm_M3_Pad_Via")
     )
     (path "/dfad1a44-dfe3-49b9-884d-77218a5dcb3d"
-      (reference "H4") (unit 1) (value "MountingHole_Pad") (footprint "MountingHole:MountingHole_4.3mm_M4_Pad_Via")
+      (reference "H4") (unit 1) (value "MountingHole_Pad") (footprint "MountingHole:MountingHole_3.2mm_M3_Pad_Via")
     )
     (path "/12a6ac24-c3c9-4b12-9357-5a8e95c1188b"
